File: Hardware/LED-display/LED-display.sch (KiCad schematic (older format))
At the start: 116 parts, among them J1 Conn_01x08, U1 74HC595, U2 74HC595, U3 74HC595

Commit message: Updating layout with additional headroom for pins > Updating DIP-16 footprint for easier placement > Updating resistor footprints to allow earier placement > Adding silk for connector pin names
Parts:
- C1, C3, C5: footprint Capacitors_THT:CP_Radial_D5.0mm_P2.00mm -> Capacitor_THT:CP_Radial_D5.0mm_P2.00mm
- C2, C4, C6: footprint Capacitors_THT:C_Disc_D5.1mm_W3.2mm_P5.00mm -> Capacitor_THT:C_Disc_D5.1mm_W3.2mm_P5.00mm
- R1, R10, R11, R13, R14, R15, R16, R17, R18, R2, R3, R4, R5, R6, R7, R8, R9: footprint Resistors_THT:R_Axial_DIN0207_L6.3mm_D2.5mm_P7.62mm_Horizontal -> Resistor_THT:R_Axial_DIN0207_L6.3mm_D2.5mm_P10.16mm_Horizontal
- U1, U2, U3: footprint Package_DIP:DIP-16_W10.16mm -> Package_DIP:DIP-16_W7.62mm
Changed lines of the file:
@@
 F 0 "U1" V 5490 1670 50  0000 C CNN
 F 1 "74HC595" V 5560 1770 50  0000 C CNN
-F 2 "Package_DIP:DIP-16_W10.16mm" H 5900 2210 50  0001 C CNN
+F 2 "Package_DIP:DIP-16_W7.62mm" H 5900 2210 50  0001 C CNN
 F 3 "http://www.ti.com/lit/ds/symlink/sn74hc595.pdf" H 5900 2210 50  0001 C CNN
 	1    5900 2210
@@
 F 0 "C3" H 6950 2440 50  0000 L CNN
 F 1 "1u" H 6950 2380 50  0000 L CNN
-F 2 "Capacitors_THT:CP_Radial_D5.0mm_P2.00mm" H 7120 2410 50  0001 C CNN
+F 2 "Capacitor_THT:CP_Radial_D5.0mm_P2.00mm" H 7120 2410 50  0001 C CNN
 F 3 "~" H 7120 2410 50  0001 C CNN
 	1    7120 2410
@@
 F 0 "C4" H 7280 2430 50  0000 L CNN
 F 1 "0.1u" H 7220 2370 50  0000 L CNN
-F 2 "Capacitors_THT:C_Disc_D5.1mm_W3.2mm_P5.00mm" H 7450 2410 50  0001 C CNN
+F 2 "Capacitor_THT:C_Disc_D5.1mm_W3.2mm_P5.00mm" H 7450 2410 50  0001 C CNN
 F 3 "~" H 7450 2410 50  0001 C CNN
 	1    7450 2410
@@
 F 0 "C1" H 4800 2440 50  0000 L CNN
 F 1 "1u" H 4800 2380 50  0000 L CNN
-F 2 "Capacitors_THT:CP_Radial_D5.0mm_P2.00mm" H 4970 2410 50  0001 C CNN
+F 2 "Capacitor_THT:CP_Radial_D5.0mm_P2.00mm" H 4970 2410 50  0001 C CNN
 F 3 "~" H 4970 2410 50  0001 C CNN
 	1    4970 2410
@@
 F 0 "C2" H 5130 2430 50  0000 L CNN
 F 1 "0.1u" H 5070 2370 50  0000 L CNN
-F 2 "Capacitors_THT:C_Disc_D5.1mm_W3.2mm_P5.00mm" H 5300 2410 50  0001 C CNN
+F 2 "Capacitor_THT:C_Disc_D5.1mm_W3.2mm_P5.00mm" H 5300 2410 50  0001 C CNN
 F 3 "~" H 5300 2410 50  0001 C CNN
 	1    5300 2410
@@
 F 0 "C5" H 3090 3620 50  0000 L CNN
 F 1 "1u" H 3090 3560 50  0000 L CNN
-F 2 "Capacitors_THT:CP_Radial_D5.0mm_P2.00mm" H 3260 3590 50  0001 C CNN
+F 2 "Capacitor_THT:CP_Radial_D5.0mm_P2.00mm" H 3260 3590 50  0001 C CNN
 F 3 "~" H 3260 3590 50  0001 C CNN
 	1    3260 3590
@@
 F 0 "C6" H 3420 3610 50  0000 L CNN
 F 1 "0.1u" H 3360 3550 50  0000 L CNN
-F 2 "Capacitors_THT:C_Disc_D5.1mm_W3.2mm_P5.00mm" H 3590 3590 50  0001 C CNN
+F 2 "Capacitor_THT:C_Disc_D5.1mm_W3.2mm_P5.00mm" H 3590 3590 50  0001 C CNN
 F 3 "~" H 3590 3590 50  0001 C CNN
 	1    3590 3590
@@
 F 0 "U2" V 7640 1660 50  0000 C CNN
 F 1 "74HC595" V 7710 1770 50  0000 C CNN
-F 2 "Package_DIP:DIP-16_W10.16mm" H 8050 2210 50  0001 C CNN
+F 2 "Package_DIP:DIP-16_W7.62mm" H 8050 2210 50  0001 C CNN
 F 3 "http://www.ti.com/lit/ds/symlink/sn74hc595.pdf" H 8050 2210 50  0001 C CNN
 	1    8050 2210
@@
 F 0 "R10" H 8150 3250 50  0000 C CNN
 F 1 "1K" H 8130 3180 50  0000 C CNN
-F 2 "Resistors_THT:R_Axial_DIN0207_L6.3mm_D2.5mm_P7.62mm_Horizontal" H 8050 3210 50  0001 C CNN
+F 2 "Resistor_THT:R_Axial_DIN0207_L6.3mm_D2.5mm_P10.16mm_Horizontal" H 8050 3210 50  0001 C CNN
 F 3 "~" H 8050 3210 50  0001 C CNN
 	1    8050 3210
@@
 F 0 "R9" H 7730 3250 50  0000 C CNN
 F 1 "1K" H 7730 3180 50  0000 C CNN
-F 2 "Resistors_THT:R_Axial_DIN0207_L6.3mm_D2.5mm_P7.62mm_Horizontal" H 7650 3210 50  0001 C CNN
+F 2 "Resistor_THT:R_Axial_DIN0207_L6.3mm_D2.5mm_P10.16mm_Horizontal" H 7650 3210 50  0001 C CNN
 F 3 "~" H 7650 3210 50  0001 C CNN
 	1    7650 3210
@@
 F 0 "R8" H 7330 3250 50  0000 C CNN
 F 1 "1K" H 7330 3180 50  0000 C CNN
-F 2 "Resistors_THT:R_Axial_DIN0207_L6.3mm_D2.5mm_P7.62mm_Horizontal" H 7250 3210 50  0001 C CNN
+F 2 "Resistor_THT:R_Axial_DIN0207_L6.3mm_D2.5mm_P10.16mm_Horizontal" H 7250 3210 50  0001 C CNN
 F 3 "~" H 7250 3210 50  0001 C CNN
 	1    7250 3210
@@
 F 0 "R7" H 6930 3250 50  0000 C CNN
 F 1 "1K" H 6930 3180 50  0000 C CNN
-F 2 "Resistors_THT:R_Axial_DIN0207_L6.3mm_D2.5mm_P7.62mm_Horizontal" H 6850 3210 50  0001 C CNN
+F 2 "Resistor_THT:R_Axial_DIN0207_L6.3mm_D2.5mm_P10.16mm_Horizontal" H 6850 3210 50  0001 C CNN
 F 3 "~" H 6850 3210 50  0001 C CNN
 	1    6850 3210
@@
 F 0 "R6" H 6530 3250 50  0000 C CNN
 F 1 "1K" H 6530 3180 50  0000 C CNN
-F 2 "Resistors_THT:R_Axial_DIN0207_L6.3mm_D2.5mm_P7.62mm_Horizontal" H 6450 3210 50  0001 C CNN
+F 2 "Resistor_THT:R_Axial_DIN0207_L6.3mm_D2.5mm_P10.16mm_Horizontal" H 6450 3210 50  0001 C CNN
 F 3 "~" H 6450 3210 50  0001 C CNN
 	1    6450 3210
@@
 F 0 "R5" H 6130 3250 50  0000 C CNN
 F 1 "1K" H 6130 3180 50  0000 C CNN
-F 2 "Resistors_THT:R_Axial_DIN0207_L6.3mm_D2.5mm_P7.62mm_Horizontal" H 6050 3210 50  0001 C CNN
+F 2 "Resistor_THT:R_Axial_DIN0207_L6.3mm_D2.5mm_P10.16mm_Horizontal" H 6050 3210 50  0001 C CNN
 F 3 "~" H 6050 3210 50  0001 C CNN
 	1    6050 3210
@@
 F 0 "R4" H 5730 3250 50  0000 C CNN
 F 1 "1K" H 5730 3180 50  0000 C CNN
-F 2 "Resistors_THT:R_Axial_DIN0207_L6.3mm_D2.5mm_P7.62mm_Horizontal" H 5650 3210 50  0001 C CNN
+F 2 "Resistor_THT:R_Axial_DIN0207_L6.3mm_D2.5mm_P10.16mm_Horizontal" H 5650 3210 50  0001 C CNN
 F 3 "~" H 5650 3210 50  0001 C CNN
 	1    5650 3210
@@
 F 0 "R3" H 5330 3250 50  0000 C CNN
 F 1 "1K" H 5330 3180 50  0000 C CNN
-F 2 "Resistors_THT:R_Axial_DIN0207_L6.3mm_D2.5mm_P7.62mm_Horizontal" H 5250 3210 50  0001 C CNN
+F 2 "Resistor_THT:R_Axial_DIN0207_L6.3mm_D2.5mm_P10.16mm_Horizontal" H 5250 3210 50  0001 C CNN
 F 3 "~" H 5250 3210 50  0001 C CNN
 	1    5250 3210
@@
 F 0 "R2" H 4930 3250 50  0000 C CNN
 F 1 "1K" H 4930 3180 50  0000 C CNN
-F 2 "Resistors_THT:R_Axial_DIN0207_L6.3mm_D2.5mm_P7.62mm_Horizontal" H 4850 3210 50  0001 C CNN
+F 2 "Resistor_THT:R_Axial_DIN0207_L6.3mm_D2.5mm_P10.16mm_Horizontal" H 4850 3210 50  0001 C CNN
 F 3 "~" H 4850 3210 50  0001 C CNN
 	1    4850 3210
@@
 F 0 "R1" H 4530 3250 50  0000 C CNN
 F 1 "1K" H 4530 3180 50  0000 C CNN
-F 2 "Resistors_THT:R_Axial_DIN0207_L6.3mm_D2.5mm_P7.62mm_Horizontal" H 4450 3210 50  0001 C CNN
+F 2 "Resistor_THT:R_Axial_DIN0207_L6.3mm_D2.5mm_P10.16mm_Horizontal" H 4450 3210 50  0001 C CNN
 F 3 "~" H 4450 3210 50  0001 C CNN
 	1    4450 3210
@@
 F 0 "U3" H 3500 5050 50  0000 C CNN
 F 1 "74HC595" H 3430 3860 50  0000 C CNN
-F 2 "Package_DIP:DIP-16_W10.16mm" H 3250 4510 50  0001 C CNN
+F 2 "Package_DIP:DIP-16_W7.62mm" H 3250 4510 50  0001 C CNN
 F 3 "http://www.ti.com/lit/ds/symlink/sn74hc595.pdf" H 3250 4510 50  0001 C CNN
 	1    3250 4510
@@
 F 0 "R13" V 9960 3560 50  0000 C CNN
 F 1 "1MEG" V 10080 3550 50  0000 C CNN
-F 2 "Resistors_THT:R_Axial_DIN0207_L6.3mm_D2.5mm_P7.62mm_Horizontal" H 10020 3550 50  0001 C CNN
+F 2 "Resistor_THT:R_Axial_DIN0207_L6.3mm_D2.5mm_P10.16mm_Horizontal" H 10020 3550 50  0001 C CNN
 F 3 "~" H 10020 3550 50  0001 C CNN
 	1    10020 3550
@@
 F 0 "R14" V 9960 3760 50  0000 C CNN
 F 1 "1MEG" V 10080 3750 50  0000 C CNN
-F 2 "Resistors_THT:R_Axial_DIN0207_L6.3mm_D2.5mm_P7.62mm_Horizontal" H 10020 3750 50  0001 C CNN
+F 2 "Resistor_THT:R_Axial_DIN0207_L6.3mm_D2.5mm_P10.16mm_Horizontal" H 10020 3750 50  0001 C CNN
 F 3 "~" H 10020 3750 50  0001 C CNN
 	1    10020 3750
@@
 F 0 "R15" V 9960 3960 50  0000 C CNN
 F 1 "1MEG" V 10080 3940 50  0000 C CNN
-F 2 "Resistors_THT:R_Axial_DIN0207_L6.3mm_D2.5mm_P7.62mm_Horizontal" H 10020 3950 50  0001 C CNN
+F 2 "Resistor_THT:R_Axial_DIN0207_L6.3mm_D2.5mm_P10.16mm_Horizontal" H 10020 3950 50  0001 C CNN
 F 3 "~" H 10020 3950 50  0001 C CNN
 	1    10020 3950
@@
 F 0 "R16" V 9960 4160 50  0000 C CNN
 F 1 "1MEG" V 10080 4150 50  0000 C CNN
-F 2 "Resistors_THT:R_Axial_DIN0207_L6.3mm_D2.5mm_P7.62mm_Horizontal" H 10020 4150 50  0001 C CNN
+F 2 "Resistor_THT:R_Axial_DIN0207_L6.3mm_D2.5mm_P10.16mm_Horizontal" H 10020 4150 50  0001 C CNN
 F 3 "~" H 10020 4150 50  0001 C CNN
 	1    10020 4150
@@
 F 0 "R17" V 9960 4370 50  0000 C CNN
 F 1 "1MEG" V 10080 4340 50  0000 C CNN
-F 2 "Resistors_THT:R_Axial_DIN0207_L6.3mm_D2.5mm_P7.62mm_Horizontal" H 10020 4350 50  0001 C CNN
+F 2 "Resistor_THT:R_Axial_DIN0207_L6.3mm_D2.5mm_P10.16mm_Horizontal" H 10020 4350 50  0001 C CNN
 F 3 "~" H 10020 4350 50  0001 C CNN
 	1    10020 4350
@@
 F 0 "R18" V 9960 4560 50  0000 C CNN
 F 1 "1MEG" V 10080 4540 50  0000 C CNN
-F 2 "Resistors_THT:R_Axial_DIN0207_L6.3mm_D2.5mm_P7.62mm_Horizontal" H 10020 4550 50  0001 C CNN
+F 2 "Resistor_THT:R_Axial_DIN0207_L6.3mm_D2.5mm_P10.16mm_Horizontal" H 10020 4550 50  0001 C CNN
 F 3 "~" H 10020 4550 50  0001 C CNN
 	1    10020 4550
@@
 F 0 "R11" H 8550 3250 50  0000 C CNN
 F 1 "1K" H 8530 3180 50  0000 C CNN
-F 2 "Resistors_THT:R_Axial_DIN0207_L6.3mm_D2.5mm_P7.62mm_Horizontal" H 8450 3210 50  0001 C CNN
+F 2 "Resistor_THT:R_Axial_DIN0207_L6.3mm_D2.5mm_P10.16mm_Horizontal" H 8450 3210 50  0001 C CNN
 F 3 "~" H 8450 3210 50  0001 C CNN
 	1    8450 3210
